File: USB_Hub_Schematic.kicad_sch (KiCad schematic)
At the start: 17 parts, among them U1 USB2517 Chip, U2 USB to microSD, U4 USB-A F, U6 USB-A F

Commit message: Schematic work
Parts:
- added C1: 0.1uF, symbol Device:C
- added C10, C6: 10 UF, symbol Device:C
- added C11, C7: 10 uF, symbol Device:C
- added C12, C8: 120 pF, symbol Device:C
- added C13, C14, C2, C3: 10 pF, symbol Device:C
- added C15: 0.1 uF, symbol Device:C
- added C16, C17, C18, C19: 33 uF, symbol Device:C
- added C4: 1 uF, symbol Device:C
- added C5, C9: 4.7 uF, symbol Device:C
- added FB1, FB2: FerriteBead, symbol Device:FerriteBead
- added L1, L2: 0.47 uH, symbol Device:L
- added R10: 32.5k, symbol Device:R
- added R11, R13, R15, R24, R25, R27, R28, R29, R30, R31, R32, R33, R34, R35, R36, R37, R38, R8: 10k, symbol Device:R
- added R12, R14: 42k, symbol Device:R
- added R16, R19, R20, R21, R23, R26: 100k, symbol Device:R
- added R17: 12k, symbol Device:R
- added R18: 453k, symbol Device:R
- added R22: 200k, symbol Device:R
- added R9: 29.8k, symbol Device:R
- added U3: MUX, lcsc_easyeda:VQFN-HR-12_L2.5-W2.0-P0.50-BL, symbol lcsc_easyeda:TPS2121RUXR
- added U5: 3.3V CONV, lcsc_easyeda:VSON-6_L1.5-W1.5-P0.50-TL, symbol lcsc_easyeda:TPS62827ADMQR
- added U7: 1.8V CONV, lcsc_easyeda:VSON-6_L1.5-W1.5-P0.50-TL, symbol lcsc_easyeda:TPS62827ADMQR
- added U8: TPS2054B, lcsc_easyeda:SOP-16_L9.9-W3.9-P1.27-LS6.1-BL, symbol lcsc_easyeda:TPS2054BDR
- added X1, X2: 24MHz, lcsc_easyeda:CRYSTAL-SMD_4P-L2.0-W1.6-BL-A, symbol lcsc_easyeda:XL7EL89CKI-111YLC-24M
Connections:
- net +3V3: now also R24.2, R25.2, R34.2, R35.2, R36.2; no longer U2.14 (VDD33), U2.6 (VDD33)
- net DN_1: now also U2.3 (USB-); no longer USB1.A7 (Dn1), USB1.B7 (Dn2)
- net DN_2: now also USB1.A7 (Dn1), USB1.B7 (Dn2); no longer USB2.A7 (Dn1), USB2.B7 (Dn2)
- net DN_3: now also USB2.A7 (Dn1), USB2.B7 (Dn2); no longer U4.2
- net DN_4: now also U4.2; no longer U6.2
- net DN_5: now also U6.2; no longer U2.3 (USB-)
- net DP_1: now also U2.2 (USB+); no longer USB1.A6 (Dp1), USB1.B6 (Dp2)
- net DP_2: now also USB1.A6 (Dp1), USB1.B6 (Dp2); no longer USB2.A6 (Dp1), USB2.B6 (Dp2)
- net DP_3: now also USB2.A6 (Dp1), USB2.B6 (Dp2); no longer U4.3
- net DP_4: now also U4.3; no longer U6.3
- net DP_5: now also U6.3; no longer U2.2 (USB+)
- net GND: now also U1.19 (TEST), U1.65 (EP), C10.1, C11.1, C13.2, C14.2, C15.1, C16.1, C17.1, C18.2, C19.2, C2.2, C3.2, C4.2, C5.2, C6.1, C7.1, C9.2, R11.2, R13.1, R15.1, R17.2, R19.2, R23.2, R27.2, R28.2, R29.1, R38.2, R9.2, U3.12 (GND), U3.3 (CP2), U5.4 (GND), U7.4 (GND), U8.1 (GND), U8.5 (GND), X1.2 (GND), X1.4 (GND), X2.2 (GND), X2.4 (GND); no longer R6.1
- net at U1.13 (CFG_SEL2): now also R29.2
- net PWR4: now reaches U1.20 (PRTPWR4)
- net PWR4: now also U8.8 (~{EN4†})
- net OC4: now reaches U1.21 (OCS4_N)
- net OC4: now also R30.1, U8.9 (~{OC4})
- net OC3: now reaches U1.22 (OCS3_N)
- net OC3: now also R31.1, U8.12 (~{OC3})
- net PWR3: now reaches U1.23 (PRTPWR3)
- net PWR3: now also U8.7 (~{EN3†})
- net PWR2: now reaches U1.26 (PRTPWR2)
- net PWR2: now also U8.4 (~{EN2†})
- net OC2: now reaches U1.27 (OCS2_N)
- net OC2: now also R32.1, U8.13 (~{OC2})
- net OC1: now reaches U1.28 (OCS1_N)
- net OC1: now also R33.1, U8.16 (~{OC1})
- net PWR1: now reaches U1.29 (PRTPWR1)
- net PWR1: now also U8.3 (~{EN1†})
- net at U1.35 (OCS5_N): now also R34.1
- net at U1.37 (OCS7_N): now also R36.1
- net at U1.38 (OCS6_N): now also R35.1
- net at U1.40 (SDA/SMBDATA/NON_REM1): now also R38.1
- net at U1.41 (SCL/SMBCLK/CFG_SEL0): now also R28.1
- net at U1.42 (HS_IND/CFG_SEL1): now also R27.1
- net at U1.44 (VBUS_DET): now also R26.1
- net at U1.45 (SUSP_IND/LOCAL_PWR/NON_REM0): now also R37.1
- net at U1.54 (USBDN6_DP/PRT_DIS_P6): now also R25.1
- net at U1.56 (USBDN7_DP/PRT_DIS_P7): now also R24.1
- net IC_X_OUT: now reaches U1.60 (XTAL2)
- net IC_X_OUT: now also C14.1, X2.3
- net IC_X_IN: now reaches U1.61 (XTAL1/CLKIN)
- net IC_X_IN: now also C13.1, X2.1
- net at U1.63 (RBIAS): now also R17.1
- net at U2.18 (RESET_N): now also R8.2
- net 3.3V_GLOBAL: now reaches U2.22 (VDD33)
- net 3.3V_GLOBAL: now also R6.1, U2.14 (VDD33), U2.6 (VDD33), C1.1, C6.2, C7.2, C8.1, C8.2, FB1.2, L1.2, R18.1, R18.2, R19.1, R20.1, R30.2, R31.2, R32.2, R33.2, U5.3 (FB)
- net X_OUT: now reaches U2.32 (XTAL2)
- net X_OUT: now also C2.1, X1.3
- net X_IN: now reaches U2.33 (XTAL1(CLKIN))
- net X_IN: now also C3.1, X1.1
- net at U2.34 (VDD18PLL): now also FB2.1
- net at U2.36 (VDDA33): now also FB1.1
- net +1V8 renamed 1.8V_GLOBAL
- net 1.8V_GLOBAL: now also C10.2, C11.2, C12.1, C12.2, FB2.2, L2.2, R21.1, R22.1, R22.2, R23.1, U7.3 (FB)
- removed net +5V: U4.1, U6.1, USB1.A4B9 (VBUS), USB1.B4A9 (VBUS), USB2.A4B9 (VBUS), USB2.B4A9 (VBUS), USB3.1 (VCC), USB4.10 (V), USB4.15 (V), USB4.2 (V), USB4.7 (V)
- new net: R9.1, U3.10 (ILM)
- new net: C4.1, U3.11 (SS)
- new net: R14.1, R15.2, U3.4 (OV2)
- new net: R12.1, R13.2, U3.5 (OV1)
- new net: R16.1, U3.9 (ST)
- new net: L2.1, U7.5 (SW)
- new net: L1.1, U5.5 (SW)
- new net: C1.2, R8.1
- new net 5V_OUT: C15.2, C5.1, C9.1, R26.2, U3.1 (OUT), U3.8 (OUT), U5.1 (EN), U5.6 (VIN), U7.1 (EN), U7.6 (VIN), U8.2 (IN1), U8.6 (IN2)
- new net HYS: R10.2, R11.1, R16.2, U3.6 (PR1)
- new net PORT1: C16.2, U8.15 (OUT1), USB1.A4B9 (VBUS), USB1.B4A9 (VBUS)
- new net PORT2: C17.2, U8.14 (OUT2), USB2.A4B9 (VBUS), USB2.B4A9 (VBUS)
- new net PORT3: C18.1, U4.1, U8.11 (OUT3)
- new net PORT4: C19.1, U6.1, U8.10 (OUT4)
- new net VBUSA: R14.2, U3.2 (IN2), USB3.1 (VCC)
- new net VBUSC: R10.1, R12.2, U3.7 (IN1), USB4.10 (V), USB4.15 (V), USB4.2 (V), USB4.7 (V)
- new net V_PG: R20.2, R21.2, U5.2 (PG), U7.2 (PG)
- no-connect marks 20 -> 39

Commit message: Schematic draft complete
Parts:
- removed C13: 10 pF, symbol Device:C
- removed R34: 10k, symbol Device:R
- added C20, C22: 1 uF, symbol Device:C
- added C21: 10 pF, symbol Device:C
- added D2, D3, D4, D5, D6, D7, D8, D9: LED, symbol Device:LED
- added FB3: FerriteBead, symbol Device:FerriteBead
- added Q2, Q3, Q4, Q5: BSS84_C114481, lcsc_easyeda:SOT-23-3_L2.9-W1.6-P1.90-LS2.8-BR, symbol lcsc_easyeda:BSS84_C114481
- added R39, R40: 330, symbol Device:R
- added R41: 10k, symbol Device:R
- added R42, R43, R44, R45: 1k, symbol Device:R
- R35, R36: value 10k -> 330
Connections:
- net PORT1 is gone; now on net PORT2: C16.2, U8.15 (OUT1), USB1.A4B9 (VBUS), USB1.B4A9 (VBUS)
- net V_PG is gone; now on net GND: R20.2, R21.2, U5.2 (PG), U7.2 (PG)
- net 3.3V_GLOBAL: now also R24.2, R25.2, R37.2, U1.24 (VDD33CR), U1.46 (VDD33), FB3.2, Q2.2 (S), Q3.2 (S), Q4.2 (S), Q5.2 (S), R41.2
- net GND: now also R35.2, R36.2, C20.2, C21.2, C22.2, D6.1 (K), D7.1 (K), D8.1 (K), D9.1 (K), R39.2, R40.2
- net IC_X_IN: now also C21.1
- net OC2: now also R33.1, U8.16 (~{OC1}), Q2.1 (G); no longer R32.1, U8.13 (~{OC2})
- net OC3: now also R32.1, U8.13 (~{OC2}), Q3.1 (G); no longer R31.1, U8.12 (~{OC3})
- net OC4: now also R31.1, U8.12 (~{OC3}), Q4.1 (G); no longer R30.1, U8.9 (~{OC4})
- net PORT2: now also R42.1; no longer C17.2, U8.14 (OUT2), USB2.A4B9 (VBUS), USB2.B4A9 (VBUS)
- net PORT3: now also C17.2, U8.14 (OUT2), USB2.A4B9 (VBUS), USB2.B4A9 (VBUS), R43.1; no longer C18.1, U4.1, U8.11 (OUT3)
- net PORT4: now also C18.1, U4.1, U8.11 (OUT3), R44.1; no longer C19.1, U6.1, U8.10 (OUT4)
- net PWR2: now also U8.3 (~{EN1†}); no longer U8.4 (~{EN2†})
- net PWR3: now also U8.4 (~{EN2†}); no longer U8.7 (~{EN3†})
- net PWR4: now also U8.7 (~{EN3†}); no longer U8.8 (~{EN4†})
- net VBUSC: no longer USB4.7 (V)
- net at R35.1: now also D2.1 (K); no longer U1.38 (OCS6_N)
- net at R36.1: now also D3.1 (K); no longer U1.37 (OCS7_N)
- net at U1.10 (VDDA33): now also U1.5 (VDDA33), U1.52 (VDDA33), U1.57 (VDDA33), U1.64 (VDD33PLL), FB3.1
- net at U1.25 (VDD18): now also C20.1
- net PWR5: now reaches U1.30 (PRTPWR5)
- net PWR5: now also U8.8 (~{EN4†})
- net OC5: now reaches U1.35 (OCS5_N)
- net OC5: now also R30.1, U8.9 (~{OC4}), Q5.1 (G)
- net at U1.43 (RESET_N): now also R41.1
- net at U1.62 (VDD18PLL): now also C22.1
- removed net +3V3: R24.2, R25.2, R35.2, R36.2
- removed net OC1: R33.1, U1.28 (OCS1_N), U8.16 (~{OC1})
- net PWR1: no longer names the net of U1.29 (PRTPWR1)
- net PWR1: no longer U8.3 (~{EN1†})
- new net: D5.2 (A), Q5.3 (D)
- new net: D5.1 (K), R40.1
- new net: D2.2 (A), Q2.3 (D)
- new net: D7.2 (A), R43.2
- new net: D4.1 (K), R39.1
- new net: D4.2 (A), Q4.3 (D)
- new net: D3.2 (A), Q3.3 (D)
- new net: D9.2 (A), R45.2
- new net: D8.2 (A), R44.2
- new net: D6.2 (A), R42.2
- new net PORT5: C19.1, R45.1, U6.1, U8.10 (OUT4)
- no-connect marks 39 -> 42
Other:
- moved on the sheet: FB1, FB2

Commit message: Schematic checks
Parts:
- removed C12: 120 pF, symbol Device:C
- removed C17: 33 uF, symbol Device:C
- removed FB2, FB3: FerriteBead, symbol Device:FerriteBead
- removed L2: 0.47 uH, symbol Device:L
- removed R1, R2, R3, R4: 5.1k, Resistor_SMD:R_01005_0402Metric, symbol Device:R
- removed R21: 100k, symbol Device:R
- removed U7: 1.8V CONV, lcsc_easyeda:VSON-6_L1.5-W1.5-P0.50-TL, symbol lcsc_easyeda:TPS62827ADMQR
- removed USB2: USB-C FEMALE, lcsc_easyeda:USB-C-SMD_TYPE-C-16PIN-2MD-073, symbol lcsc_easyeda:TYPE-C16PIN2MD
- added C23, C24, C25, C29, C32, C36: 0.1 uF, symbol Device:C
- added C26, C27, C30, C31, C35: 1 uF, symbol Device:C
- added C28: 10 uF, symbol Device:C
- added C34: 33 uF, symbol Device:C
- added R34, R47: 100k, symbol Device:R
- added R46: 10k, symbol Device:R
- added R48: 1M, symbol Device:R
- added R49, R50, R52: 36k, Resistor_SMD:R_01005_0402Metric, symbol Device:R
- added R51: 330, symbol Device:R
- added U10, U11, U12, U13, U14, U15, U9: TP, lcsc_easyeda:TEST-SMD_L2.7-W1.0, symbol lcsc_easyeda:5015
- added USB5: USB-C FEMALE, lcsc_easyeda:USB-C-SMD_TYPE-C-16PIN-2MD-073, symbol lcsc_easyeda:TYPE-C16PIN2MD
- C10: value 10 UF -> 0.1 uF
- C11: value 10 uF -> 0.1 uF
- C9: value 4.7 uF -> 0.1 uF
- R22: value 200k -> 330
- R23: value 100k -> 36k; footprint (none) -> Resistor_SMD:R_01005_0402Metric
- R26: value 100k -> 10k
Connections:
- net 3.3V_GLOBAL: now also R23.1, R26.2, C30.1, C31.1, C32.1, C35.1, C36.1, R46.2, R49.1, R50.1, R52.1, U10.1
- net 5V_OUT: now also C28.1, R34.2, U9.1; no longer C9.1, R26.2
- net DN_3: now also USB5.A7 (Dn1), USB5.B7 (Dn2)
- net DP_3: now also USB5.A6 (Dp1), USB5.B6 (Dp2)
- net GND: now also C3.1, R22.1, C23.2, C24.1, C25.2, C26.2, C27.1, C28.2, C29.2, C30.2, C32.2, C34.1, C35.2, C36.2, R47.1, R51.1, USB5.A1B12 (GND), USB5.B1A12 (GND); no longer C3.2, R23.2, USB1.13 (EH), USB1.14 (EH)
- net IC_X_OUT: now also R48.2
- net PORT3: now also C34.2, USB5.A4B9 (VBUS), USB5.B4A9 (VBUS)
- net VBUSC: now also USB4.7 (V)
- net X_IN: now also C3.2; no longer C3.1
- net TP_SUSPIND: now reaches R37.1, U1.45 (SUSP_IND/LOCAL_PWR/NON_REM0)
- net TP_SUSPIND: now also U13.1
- net at U1.10 (VDDA33), U1.5 (VDDA33), U1.52 (VDDA33)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: now also C9.1, C23.1, C25.1, C29.1, C31.2; no longer U1.64 (VDD33PLL)
- net at U2.34 (VDD18PLL): now also C26.1
- net at USB1.A5 (CC1): now also R49.2
- net TP_RESET: now reaches R41.1, U1.43 (RESET_N)
- net TP_RESET: now also U15.1
- net at R26.1: now also U1.55 (USBDN7_DM/PRT_DIS_M7); no longer U1.44 (VBUS_DET)
- net at U1.53 (USBDN6_DM/PRT_DIS_M6): now also R46.1
- net TP_18PLL: now reaches C22.1, U1.62 (VDD18PLL)
- net TP_18PLL: now also U12.1
- net at USB1.B5 (CC2): now also R23.2
- removed net 1.8V_GLOBAL: C10.2, C11.2, R22.1, R22.2, R23.1, U2.13 (VDD18)
- net IC_X_IN renamed 1M
- net 1M: now also R48.1
- new net: R50.2, USB5.A5 (CC1)
- new net: C11.2, R51.2, USB5.13 (EH), USB5.14 (EH)
- new net: C27.2, U2.13 (VDD18)
- new net: C10.2, R22.2, USB1.13 (EH), USB1.14 (EH)
- new net: R52.2, USB5.B5 (CC2)
- new net TP_33PLL: C24.2, U1.64 (VDD33PLL), U11.1
- new net TP_VBUS: R34.1, R47.2, U1.44 (VBUS_DET), U14.1
- no-connect marks 42 -> 40
Other:
- moved on the sheet: FB1
