File: USB_Hub_Schematic.kicad_sch (KiCad schematic)
At the start: 114 parts, among them J1 USB-C, J2 USB-A, U1 USB2517 Chip, U10 TP, U11 TP, U12 TP, U13 TP, U14 TP, U15 TP, U16 TPS25821, U17 TPS25821, U3 MUX, U4 USB to microSD, U7 TPS2052B, U8 3.3V CONV, U9 TP, X3 24MHz Osc

Commit message: Routing continued
Parts:
- removed C15, C16, C21: 10 uF, Capacitor_SMD:C_0805_2012Metric, symbol Device:C
- removed C26: 100 pF, Capacitor_SMD:C_0402_1005Metric, symbol Device:C
- removed C6: 4.7 uF, Capacitor_SMD:C_0603_1608Metric, symbol Device:C
- removed L2: 0.47 uH, Inductor_SMD:L_1008_2520Metric, symbol Device:L
- removed R20: 453k, Resistor_SMD:R_0603_1608Metric, symbol Device:R
- removed R22: 100k, Resistor_SMD:R_0603_1608Metric, symbol Device:R
- removed R50, R58: 10k, Resistor_SMD:R_0603_1608Metric, symbol Device:R
- removed U8: 3.3V CONV, lcsc_easyeda:VSON-6_L1.5-W1.5-P0.50-TL, symbol lcsc_easyeda:TPS62827ADMQR
- added C2: 0.1 uF, Capacitor_SMD:C_0402_1005Metric, symbol Device:C
- added C3: 47 uF, Capacitor_SMD:C_0805_2012Metric, symbol Device:C
- added R6: 33k, Resistor_SMD:R_0603_1608Metric, symbol Device:R
- added R7: 68k, Resistor_SMD:R_0603_1608Metric, symbol Device:R
- added U2: 3.3V CONV, lcsc_easyeda:QFN-7_L4.0-W3.3_TPSM863257RDXR, symbol lcsc_easyeda:TPSM863253RDXR
Connections:
- net 3.3V_GLOBAL: now also C3.1, U2.3 (VOUT), U2.7 (VOS)
- net 5V_OUT: now also C2.1, R7.2, U2.1 (VIN); no longer U16.3 (CHG), U17.3 (CHG)
- net GND: now also U16.3 (CHG), U17.3 (CHG), C2.2, C3.2, R6.2, U2.4 (PGND)
- new net: R6.1, R7.1, U2.6 (EN)
- no-connect marks 23 -> 26
