File: USB_Hub_Schematic.kicad_sch (KiCad schematic)
At the start: 108 parts, among them J1 USB-C, J2 USB-A, U1 USB2517 Chip, U10 TP, U11 TP, U12 TP, U13 TP, U14 TP, U15 TP, U16 TPS25821, U17 TPS25821, U2 3.3V CONV, U3 MUX, U4 USB to microSD, U7 TPS2052B, U9 TP, X3 24MHz Osc

Commit message: Routing draft complete
Parts:
- removed C50: 33 uF, Capacitor_SMD:C_0805_2012Metric, symbol Device:C
- removed C51: 0.1 uF, Capacitor_SMD:C_0402_1005Metric, symbol Device:C
- removed R35: 330, Resistor_SMD:R_0603_1608Metric, symbol Device:R
- removed USB1, USB2: USB-C F, lcsc_easyeda:USB-C-SMD_GT-USB-7100A, symbol lcsc_easyeda:GT-USB-7100A
- added C21: 33 uF, Capacitor_SMD:C_0805_2012Metric, symbol Device:C
- added C26: 0.1 uF, Capacitor_SMD:C_0402_1005Metric, symbol Device:C
- added R33: 330, Resistor_SMD:R_0603_1608Metric, symbol Device:R
- added USB3, USB4: USB-C F, lcsc_easyeda:USB-C-SMD_MC-403L68-Z20, symbol lcsc_easyeda:MC-403L68-Z20
Connections:
- net C1_CC1: now also USB3.A5 (CC1)
- net C1_CC2: now also USB3.B5 (CC2)
- net C2_CC1: now also USB4.A5 (CC1)
- net C2_CC2: now also USB4.B5 (CC2)
- net DN_2: now also USB3.A7 (DN1)
- net DN_3: now also USB4.A7 (DN1)
- net DP_2: now also USB3.A6 (DP1)
- net DP_3: now also USB4.A6 (DP1)
- net GND: now also C21.1, C26.2, R33.2, USB3.B1 (GND), USB3.B12 (GND), USB4.B1 (GND), USB4.B12 (GND)
- net PORT2: now also USB3.B4 (VBUS), USB3.B9 (VBUS)
- net PORT3: now also C21.2, USB4.B4 (VBUS), USB4.B9 (VBUS)
- net at C18.1, R32.1: now also USB3.10 (EH), USB3.11 (EH), USB3.12 (EH), USB3.9 (EH)
- new net: C26.1, R33.1, USB4.10 (EH), USB4.11 (EH), USB4.12 (EH), USB4.9 (EH)

Commit message: Routing Updates
Parts:
- removed R24, R25, R26, R42, R46: 10k, Resistor_SMD:R_0603_1608Metric, symbol Device:R
- added C5: 1 uF, Capacitor_SMD:C_0603_1608Metric, symbol Device:C
- added U18, U19: TP, lcsc_easyeda:TEST-SMD_L2.7-W1.0, symbol lcsc_easyeda:5015
- added U5: 24AA02, lcsc_easyeda:SOT-23-5_L2.9-W1.6-P0.95-LS2.8-BL-3, symbol lcsc_easyeda:24AA02T-I_OT
Connections:
- net 3.3V_GLOBAL: now also R27.2, C5.1, U5.4 (VCC)
- net GND: now also C5.2, U5.2 (VSS), U5.5 (WP); no longer R27.2, R28.2, R38.2
- new net EEPROM_CLK: R28.2, U18.1, U5.1 (SCL)
- new net EEPROM_DATA: R38.2, U19.1, U5.3 (SDA)
- no-connect marks 26 -> 30

Commit message: PCBWay Order Sent
Parts:
- C1, C20, C22, C31, C35, C4, C5: LCSC Part (none) -> C15849
- C12, C13, C17, C3, C33, C38, C39: LCSC Part (none) -> C16780
- C18, C2, C23, C24, C25, C26, C29, C32, C36, C37, C40, C41, C42, C44, C9: LCSC Part (none) -> C1525
- C19, C21, C30, C48: LCSC Part (none) -> C342635
- C28: LCSC Part (none) -> C19666
- C43, C45: LCSC Part (none) -> C15008
- D10, D13, D14, D15, D2: LCSC Part (none) -> C2290
- D11, D12, D16, D17: LCSC Part (none) -> C2286
- R1, R16, R2, R34, R47, R49, R51, R54, R56: LCSC Part (none) -> C25803
- R10, R6: LCSC Part (none) -> C4216
- R11, R13, R15, R27, R28, R29, R3, R38, R4, R41: LCSC Part (none) -> C177337
- R12, R14, R9: LCSC Part (none) -> C861392
- R17: LCSC Part (none) -> C22790
- R21, R23, R30, R31, R5, R52, R53, R55, R57: LCSC Part (none) -> C177649
- R32, R33: LCSC Part (none) -> C23138
- R7: LCSC Part (none) -> C22356449
