File: USB_Hub_Schematic.kicad_pcb (KiCad board)
At the start: 4 copper layers, 43.9 x 87.6 mm, 108 parts, among them J1 USB-C, J2 USB-A, U1 USB2517 Chip, U10 TP, U11 TP, U12 TP, U13 TP, U14 TP, U15 TP, U16 TPS25821, U17 TPS25821, U2 3.3V CONV, U3 MUX, U4 USB to microSD, U7 TPS2052B, U9 TP, X3 24MHz Osc

Commit message: Routing draft complete
Parts:
- removed C50: 33 uF, Capacitor_SMD:C_0805_2012Metric
- removed C51: 0.1 uF, Capacitor_SMD:C_0402_1005Metric
- removed R35: 330, Resistor_SMD:R_0603_1608Metric
- removed USB1, USB2: USB-C F, lcsc_easyeda:USB-C-SMD_GT-USB-7100A
- added C21: 33 uF, Capacitor_SMD:C_0805_2012Metric, F.Cu at (154.9, 64.7)
- added C26: 0.1 uF, Capacitor_SMD:C_0402_1005Metric, F.Cu at (158.5, 64.5)
- added R33: 330, Resistor_SMD:R_0603_1608Metric, F.Cu at (157.2, 64.0)
- added USB3: USB-C F, lcsc_easyeda:USB-C-SMD_MC-403L68-Z20, F.Cu at (160.8, 86.8)
- added USB4: USB-C F, lcsc_easyeda:USB-C-SMD_MC-403L68-Z20, F.Cu at (160.7, 70.6)
- moved C17 4.06 mm to (151.9, 64.3)
- moved C39 4.06 mm to (156.0, 64.3)
- moved D2 1.02 mm to (137.4, 104.9)
- moved R54 0.11 mm to (150.9, 65.3)
- moved D12 0.10 mm to (150.1, 63.0)
- moved R53 0.10 mm to (151.6, 63.0)
- moved R2 0.06 mm to (155.4, 69.8)
Routing:
- net /3.3V_GLOBAL: track 79.5 -> 296.6 mm
- net /5V_OUT: track 76.1 -> 264.6 mm, vias 11 -> 12
- net /VBUSA: track 11.5 -> 60.1 mm, vias 4 -> 2
- net Net-(C26-Pad1): track 0.00 -> 20.4 mm
- net GND: track 327.5 -> 346.8 mm
- net Net-(C18-Pad1): track 3.20 -> 20.2 mm
- net /VBUSC: track 16.0 -> 25.3 mm, vias 4 -> 2
- net Net-(C23-Pad1): track 23.0 -> 31.8 mm
- net /PORT2: track 17.3 -> 11.9 mm, vias 2 -> 0
- net /PORT3: track 17.4 -> 13.7 mm, vias 2 -> 0
- net Net-(C51-Pad1): track 3.19 -> 0.00 mm
- net /C2_CC1: track 14.8 -> 17.0 mm
- net /OC2: track 45.8 -> 47.7 mm
- net /C1_CC1: track 13.0 -> 14.7 mm
- net /DP_2: track 32.7 -> 34.3 mm
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- added copper zone on In2.Cu, net /3.3V_GLOBAL
- added copper zone on In2.Cu, net /5V_OUT
- added copper zone on In2.Cu, net /VBUSA
- added copper zone on In2.Cu, net /VBUSC
- added copper zone on In1.Cu, net GND
Other:
- board size 43.9 x 87.6 mm -> 43.5 x 88 mm
